File: 2026_InClass_2Wheel_Robot_Donnellan/.history/2026_InClass_2Wheel_Robot_Donnellan.kicad_pcb (KiCad board)
At the start: 2 copper layers, 55 x 55 mm, 57 parts, among them J1 BATT_CONN, J2 M1_CONN, J3 M2_CONN, J4 Conn_01x08, J5 Conn_02x04_Odd_Even, J6 ENCODER_CONN, J7 ENCODER_CONN, J8 MT6701_CONN, J9 USB_C_Receptacle_USB2.0_14P, SW1 SW_uP_Reset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

Commit message: Revised PCB design
Parts:
- added H1: Mount 1, MountingHole:MountingHole_2.1mm, F.Cu at (66.5, 155.8)
- added H2: Mount 2, MountingHole:MountingHole_2.1mm, F.Cu at (114.7, 155.8)
- C16: footprint Capacitor_SMD:C_0805_2012Metric_Pad1.18x1.45mm_HandSolder -> Capacitor_Tantalum_SMD:CP_EIA-6032-28_Kemet-C_HandSolder
- moved C16 2.02 mm to (74.5, 149.1)
Routing:
- net GND: track 57.3 -> 58.3 mm
- net VM: track 45.2 -> 45.8 mm
